File: PROJECT.sch (KiCad schematic (older format))
At the start: 25 parts

Commit message: PCB
Parts:
- removed C? (x2): C_Small, symbol device:C_Small
- C1, C2, C3, C4, C5, C6: renamed from C?; footprint (none) -> Capacitor_SMD:C_0805_2012Metric
- Q1: renamed from Q?; footprint (none) -> Keebio-Parts:SOT-23_Handsoldering
- SPI1: footprint (none) -> Connector_PinHeader_2.00mm:PinHeader_2x03_P2.00mm_Vertical; symbol conn:Conn_02x03_Counter_Clockwise -> PROJECT-rescue:Conn_02x03_Counter_Clockwise-conn
- SW1: renamed from SW?; footprint (none) -> Button_Switch_SMD:SW_SPST_SKQG_WithoutStem
- U1: renamed from U?; footprint (none) -> Mixed Lib:SOT143B
- U2: renamed from U?; footprint (none) -> keyboard_parts:QFP44; symbol atmel:ATmega32U4 -> PROJECT-rescue:ATmega32U4-atmel
- USB1: renamed from USB?; footprint (none) -> Type-C:HRO-TYPE-C-31-M-12
- USBCap1: footprint (none) -> Capacitor_SMD:C_0805_2012Metric
- X1: renamed from X?; footprint (none) -> Mixed Lib:CSTCE
- gave numbers to parts that had none: 3
Connections:
- wire segments 118 -> 124
Other:
- moved on the sheet: X1

Commit message: PCB design
Parts:
- C1: value C -> 4.7uf
- C6: value C -> 1uf
Connections:
- net GND: now also X1.2; no longer X1.3
- net at U2.16 (XTAL2): now also X1.3; no longer X1.2
Other:
- moved on the sheet: X1
Changed lines of the file:
@@
 P 19600 12200
 F 0 "C1" H 19715 12246 50  0000 L CNN
-F 1 "C" H 19715 12155 50  0000 L CNN
+F 1 "4.7uf" H 19715 12155 50  0000 L CNN
 F 2 "Capacitor_SMD:C_0805_2012Metric" H 19638 12050 50  0001 C CNN
 F 3 "~" H 19600 12200 50  0001 C CNN
@@
 P 21350 13050
 F 0 "C6" V 21098 13050 50  0000 C CNN
-F 1 "C" V 21189 13050 50  0000 C CNN
+F 1 "1uf" V 21189 13050 50  0000 C CNN
 F 2 "Capacitor_SMD:C_0805_2012Metric" H 21388 12900 50  0001 C CNN
 F 3 "~" H 21350 13050 50  0001 C CNN
@@
 L keyboard_parts:XTAL_GND X1
 U 1 1 5BBBD0FA
-P 21325 14100
-F 0 "X1" H 21325 14392 60  0000 C CNN
-F 1 "XTAL_GND" H 21325 14286 60  0000 C CNN
-F 2 "Mixed Lib:CSTCE" H 21325 14100 60  0001 C CNN
-F 3 "" H 21325 14100 60  0000 C CNN
-	1    21325 14100
-	0    1    1    0
-$EndComp
-Wire Wire Line
-	21125 14100 21075 14100
-$Comp
-L power:GND #PWR0107
-U 1 1 5BBBFFA0
-P 21075 14100
-F 0 "#PWR0107" H 21075 13850 50  0001 C CNN
-F 1 "GND" H 21080 13927 50  0000 C CNN
-F 2 "" H 21075 14100 50  0001 C CNN
-F 3 "" H 21075 14100 50  0001 C CNN
-	1    21075 14100
+P 21225 14100
+F 0 "X1" H 21225 14392 60  0000 C CNN
+F 1 "XTAL_GND" H 21225 14286 60  0000 C CNN
+F 2 "Mixed Lib:CSTCE" H 21225 14100 60  0001 C CNN
+F 3 "" H 21225 14100 60  0000 C CNN
+	1    21225 14100
 	0    1    1    0
 $EndComp
@@
 $EndSheet
 Wire Wire Line
-	21325 13800 21675 13800
-Wire Wire Line
 	21675 13800 21675 14050
 Wire Wire Line
@@
 	21900 14150 21675 14150
 Wire Wire Line
-	21675 14150 21675 14400
-Wire Wire Line
-	21675 14400 21325 14400
+	21225 14400 21225 14450
+$Comp
+L power:GND #PWR0107
+U 1 1 5BBBFFA0
+P 21225 14450
+F 0 "#PWR0107" H 21225 14200 50  0001 C CNN
+F 1 "GND" H 21230 14277 50  0000 C CNN
+F 2 "" H 21225 14450 50  0001 C CNN
+F 3 "" H 21225 14450 50  0001 C CNN
+	1    21225 14450
+	1    0    0    -1
+$EndComp
+Wire Wire Line
+	21675 14150 21675 14350
+Wire Wire Line
+	21675 14350 21025 14350
+Wire Wire Line
+	21025 14350 21025 14100
+Wire Wire Line
+	21225 13800 21675 13800
 $EndSCHEMATC

Commit message: Update
Connections:
- net LEDVCC is gone; now on an unnamed net: Q1.2 (C)
- net +5V: no longer Q1.3 (E)
- net GND: now also Q1.1 (B)
- net at NPNR1.1: no longer Q1.1 (B)
- new net LEDGND: Q1.3 (E)
Other:
- moved on the sheet: NPNR1
Changed lines of the file:
@@
 L device:R NPNR1
 U 1 1 5BC33255
-P 24650 11350
-F 0 "NPNR1" V 24550 11350 50  0000 C CNN
-F 1 "1.5k" V 24650 11350 50  0000 C CNN
-F 2 "" V 24580 11350 50  0001 C CNN
-F 3 "~" H 24650 11350 50  0001 C CNN
-	1    24650 11350
+P 25100 11050
+F 0 "NPNR1" V 25000 11050 50  0000 C CNN
+F 1 "1.5k" V 25100 11050 50  0000 C CNN
+F 2 "" V 25030 11050 50  0001 C CNN
+F 3 "~" H 25100 11050 50  0001 C CNN
+	1    25100 11050
 	0    1    1    0
 $EndComp
 Wire Wire Line
-	24500 11350 24375 11350
-Text GLabel 24375 11350 0    50   Input ~ 0
+	24950 11050 24825 11050
+Text GLabel 24825 11050 0    50   Input ~ 0
 LEDPWM
-Text GLabel 25250 11050 0    50   Input ~ 0
-LEDVCC
+Text GLabel 25250 11650 0    50   Input ~ 0
+LEDGND
 Wire Wire Line
 	25250 11650 25250 11550
@@
 Wire Wire Line
 	19925 12050 20225 12050
-$Comp
-L keyboard_parts:+5V #PWR0116
-U 1 1 5C2A869E
-P 25250 11650
-F 0 "#PWR0116" H 25250 11620 20  0001 C CNN
-F 1 "+5V" V 25250 11757 30  0000 L CNN
-F 2 "" H 25250 11650 60  0000 C CNN
-F 3 "" H 25250 11650 60  0000 C CNN
-	1    25250 11650
-	0    1    1    0
-$EndComp
 $Sheet
 S 25475 14850 2425 1200
@@
 Wire Wire Line
 	21225 13800 21675 13800
+$Comp
+L power:GND #PWR?
+U 1 1 5D35752A
+P 24800 11350
+F 0 "#PWR?" H 24800 11100 50  0001 C CNN
+F 1 "GND" H 24805 11177 50  0000 C CNN
+F 2 "" H 24800 11350 50  0001 C CNN
+F 3 "" H 24800 11350 50  0001 C CNN
+	1    24800 11350
+	1    0    0    -1
+$EndComp
 $EndSCHEMATC
